Commit message: cao_size1
change the origin xyz of base_link

File: install/cpp06_urdf/share/cpp06_urdf/urdf/xacro/car_base.urdf.xacro (robot description, xacro)
@@ -39,5 +39,5 @@
         </geometry>
         <material name="yellow"/>
-        <origin xyz="0.0 0.0 ${car_height/2 + distance}"/>
+        <origin xyz="0.0 0.0 0.1275"/>
     </visual>
 </link>
